Commit message: worked 2 cameras with tello model

File: urdf/model.xacro (robot description, xacro)
@@ -2,23 +2,52 @@
 <robot name="mascot" xmlns:xacro="http://www.ros.org/wiki/xacro">
   <xacro:property name="robot_name" value="$(arg robot_name)" />
+  <material name="red">
+    <color rgba="1 0 0 1"/>
+  </material>
   <link name="${robot_name}_base_link">
     <inertial>
       <mass value="1.477" />
-      <origin rpy="0 0 0" xyz="0 0 0" />
+      <origin rpy="1.57 0 0" xyz="0 0 0" />
       <inertia ixx="0.1152" ixy="0" ixz="0" iyy="0.1152" iyz="0" izz="0.218" />
     </inertial>
     <collision name="mascot__collision">
-      <origin rpy="0 0 0" xyz="0   0   0.04" />
+      <origin rpy="1.57 0 0" xyz="0   0   0.04" />
       <geometry>
-        <mesh filename="package://mascot/meshes/quadrotor_4.stl" />
+        <mesh scale="0.001 0.001 0.001" filename="package://mascot/meshes/Dji_Tello.stl" />
       </geometry>
     </collision>
     <visual name="mascot__visual">
-      <origin rpy="0 0 0" xyz="0   0   0.04" />
+      <origin rpy="1.57 0 0" xyz="0   0   0.04" />
       <geometry>
-        <mesh filename="package://mascot/meshes/quadrotor_4.dae" />
+        <mesh scale="0.001 0.001 0.001" filename="package://mascot/meshes/Dji_Tello.dae" />
       </geometry>
     </visual>
   </link>
+  <link name="${robot_name}_down_camera_link">
+    <visual>
+        <geometry>
+            <sphere radius="0.03"/>
+        </geometry>
+        <material name="red"/>
+    </visual>
+  </link>
+  <joint name="${robot_name}_down_camera_joint" type="fixed">
+    <parent link="${robot_name}_base_link"/>
+    <child link="${robot_name}_down_camera_link"/>
+    <origin xyz="-0.12 0 -0.03" rpy="0 1.570796326794897 0"/>
+  </joint>
+  <link name="${robot_name}_front_camera_link">
+    <visual>
+        <geometry>
+            <sphere radius="0.03"/>
+        </geometry>
+        <material name="red"/>
+    </visual>
+  </link>
+  <joint name="${robot_name}_front_camera_joint" type="fixed">
+    <parent link="${robot_name}_base_link"/>
+    <child link="${robot_name}_front_camera_link"/>
+    <origin xyz="0.25 0 0.04" rpy="0 0 0"/>
+  </joint>
   <gazebo>
     <plugin name='simple_drone' filename='libplugin_drone.so'>
@@ -62,68 +91,10 @@
     </plugin>
   </gazebo>
-  <!-- Sensors -->
-  <gazebo>
-    <sensor name='sensor_imu' type='imu'>
-      <always_on> 1 </always_on>
-      <update_rate> 100 </update_rate>
-      <pose> 0 0 0 0 0 0 </pose>
-      <plugin name='ros_imu' filename='libplugin_ros_imu.so'></plugin>
-      <imu>
-        <noise>
-          <type>gaussian</type>
-          <rate>
-            <mean> 0 </mean>
-            <stddev> 0 </stddev>
-          </rate>
-          <accel>
-            <mean> 0 </mean>
-            <stddev> 0.00 </stddev>
-          </accel>
-        </noise>
-      </imu>
-    </sensor>
-    <!-- Sonar sensor in 100fps -->
-    <sensor name='sensor_sonar' type='sonar'>
-      <always_on>1</always_on>
-      <visualize>0</visualize>
-      <update_rate>100</update_rate>
-      <pose> 0.5 0 0.3 0 1.570796327 3.141592653 </pose>
-      <plugin name='ros_sonar' filename='libplugin_ros_sonar.so'></plugin>
-      <sonar>
-        <min>0</min>
-        <max>5</max>
-        <radius>1.33974596</radius>
-      </sonar>
-    </sensor>
-    <!-- front camera -->
-    <sensor name="front_camera" type="camera">
-      <camera>
-        <horizontal_fov>1.5</horizontal_fov>
-        <image>
-          <width>640</width>
-          <height>480</height>
-          <format>R8G8B8</format>
-        </image>
-        <clip>
-          <near>0.1</near>
-          <far>100</far>
-        </clip>
-        <noise>
-          <type>gaussian</type>
-          <mean>0.0</mean>
-          <stddev>0.005</stddev>
-        </noise>
-      </camera>
-      <pose> 0.2 0.0 0.0 0 0 0 </pose>
-      <always_on>1</always_on>
-      <update_rate>60</update_rate>
+  <gazebo reference="${robot_name}_front_camera_link">
+    <sensor name="${robot_name}_front_camera" type="camera">
+      <alwaysOn>true</alwaysOn>
       <visualize>true</visualize>
-      <plugin name='front_camera' filename='libplugin_ros_cam.so'>
-        <imageTopicName>/drone/front_camera/image_raw</imageTopicName>
-      </plugin>
-    </sensor>
-    <!-- downward looking camera -->
-    <sensor name="down_camera" type="camera">
-      <camera>
+      <update_rate>15</update_rate>
+      <camera name="front">
         <horizontal_fov>1.047</horizontal_fov>
         <image>
@@ -142,11 +113,58 @@
         </noise>
       </camera>
-      <pose> 0.0 0.0 0.0 0 1.570796326794897 0 </pose>
-      <always_on>1</always_on>
+      <plugin name='${robot_name}_front_camera' filename='libgazebo_ros_camera.so'>
+        <alwaysOn>true</alwaysOn>
+        <updateRate>0.0</updateRate>
+        <cameraName>${robot_name}_front_camera</cameraName>
+        <imageTopicName>image_raw</imageTopicName>
+        <cameraInfoTopicName>camera_info</cameraInfoTopicName>
+        <frameName>${robot_name}_front_camera_link</frameName>
+        <hackBaseline>0.07</hackBaseline>
+        <distortionK1>0.0</distortionK1>
+        <distortionK2>0.0</distortionK2>
+        <distortionK3>0.0</distortionK3>
+        <distortionT1>0.0</distortionT1>
+        <distortionT2>0.0</distortionT2>
+      </plugin>
+      <frame_name>${robot_name}_front_camera_link</frame_name>
+    </sensor>
+  </gazebo>
+  <gazebo reference="${robot_name}_down_camera_link">
+    <sensor name="${robot_name}_down_camera" type="camera">
+      <alwaysOn>true</alwaysOn>
+      <visualize>true</visualize>
       <update_rate>15</update_rate>
-      <visualize>true</visualize>
-      <plugin name='down_camera' filename='libplugin_ros_cam.so'>
-        <imageTopicName>/drone/down_camera/image_raw</imageTopicName>
+      <camera name="head">
+        <horizontal_fov>1.047</horizontal_fov>
+        <image>
+          <width>640</width>
+          <height>360</height>
+          <format>R8G8B8</format>
+        </image>
+        <clip>
+          <near>0.1</near>
+          <far>100</far>
+        </clip>
+        <noise>
+          <type>gaussian</type>
+          <mean>0.0</mean>
+          <stddev>0.005</stddev>
+        </noise>
+      </camera>
+      <plugin name='${robot_name}_down_camera' filename='libgazebo_ros_camera.so'>
+        <alwaysOn>true</alwaysOn>
+        <updateRate>0.0</updateRate>
+        <cameraName>${robot_name}_down_camera</cameraName>
+        <imageTopicName>image_raw</imageTopicName>
+        <cameraInfoTopicName>camera_info</cameraInfoTopicName>
+        <frameName>${robot_name}_down_camera_link</frameName>
+        <hackBaseline>0.07</hackBaseline>
+        <distortionK1>0.0</distortionK1>
+        <distortionK2>0.0</distortionK2>
+        <distortionK3>0.0</distortionK3>
+        <distortionT1>0.0</distortionT1>
+        <distortionT2>0.0</distortionT2>
       </plugin>
+      <frame_name>${robot_name}_down_camera_link</frame_name>
     </sensor>
   </gazebo>

Commit message: with imu and sonar sensor

File: urdf/model.xacro (robot description, xacro)
@@ -12,13 +12,13 @@
     </inertial>
     <collision name="mascot__collision">
-      <origin rpy="1.57 0 0" xyz="0   0   0.04" />
+      <origin rpy="1.57 0 0" xyz="0   0   0.02" />
       <geometry>
-        <mesh scale="0.001 0.001 0.001" filename="package://mascot/meshes/Dji_Tello.stl" />
+        <mesh scale="0.0005 0.0005 0.0005" filename="package://mascot/meshes/Dji_Tello.stl" />
       </geometry>
     </collision>
     <visual name="mascot__visual">
-      <origin rpy="1.57 0 0" xyz="0   0   0.04" />
+      <origin rpy="1.57 0 0" xyz="0   0   0.02" />
       <geometry>
-        <mesh scale="0.001 0.001 0.001" filename="package://mascot/meshes/Dji_Tello.dae" />
+        <mesh scale="0.0005 0.0005 0.0005" filename="package://mascot/meshes/Dji_Tello.dae" />
       </geometry>
     </visual>
@@ -27,5 +27,5 @@
     <visual>
         <geometry>
-            <sphere radius="0.03"/>
+            <sphere radius="0.015"/>
         </geometry>
         <material name="red"/>
@@ -35,10 +35,10 @@
     <parent link="${robot_name}_base_link"/>
     <child link="${robot_name}_down_camera_link"/>
-    <origin xyz="-0.12 0 -0.03" rpy="0 1.570796326794897 0"/>
+    <origin xyz="-0.06 0 -0.015" rpy="0 1.570796326794897 0"/>
   </joint>
   <link name="${robot_name}_front_camera_link">
     <visual>
         <geometry>
-            <sphere radius="0.03"/>
+            <sphere radius="0.015"/>
         </geometry>
         <material name="red"/>
@@ -48,5 +48,5 @@
     <parent link="${robot_name}_base_link"/>
     <child link="${robot_name}_front_camera_link"/>
-    <origin xyz="0.25 0 0.04" rpy="0 0 0"/>
+    <origin xyz="0.125 0 0.02" rpy="0 0 0"/>
   </joint>
   <gazebo>
@@ -169,3 +169,41 @@
     </sensor>
   </gazebo>
+  <gazebo reference="${robot_name}_base_link">
+     <sensor name='${robot_name}_sensor_sonar' type='sonar'>
+      <always_on>1</always_on>
+      <visualize>1</visualize>
+      <update_rate>100</update_rate>
+      <pose> 0 0 0 0 0 3.141592653 </pose>
+      <plugin name='${robot_name}_sonar' filename='libplugin_ros_sonar.so'>
+         <topicName>${robot_name}_sonar_sensor</topicName>
+         <frameName>${robot_name}_down_camera_link</frameName>
+      </plugin>
+      <sonar>
+        <min>0</min>
+        <max>1</max>
+        <radius>0.13974596</radius>
+      </sonar>
+      <frame_name>${robot_name}_down_camera_link</frame_name>
+    </sensor>
+  </gazebo>
+  <gazebo reference="${robot_name}_base_link">
+    <gravity>true</gravity>
+    <sensor name="${robot_name}_imu_sensor" type="imu">
+      <always_on>true</always_on>
+      <update_rate>100</update_rate>
+      <visualize>true</visualize>
+      <topic>__default_topic__</topic>
+      <plugin filename="libgazebo_ros_imu_sensor.so" name="imu_plugin">
+        <topicName>${robot_name}_imu</topicName>
+        <bodyName>${robot_name}_base_link</bodyName>
+        <updateRateHZ>10.0</updateRateHZ>
+        <gaussianNoise>0.0</gaussianNoise>
+        <xyzOffset>0 0 0</xyzOffset>
+        <rpyOffset>0 0 0</rpyOffset>
+        <frameName>${robot_name}_base_link</frameName>
+        <initialOrientationAsReference>false</initialOrientationAsReference>
+      </plugin>
+      <pose>0 0 0 0 0 0</pose>
+    </sensor>
+  </gazebo>
 </robot>

Commit message: new model, fixed imu and physics

File: urdf/model.xacro (robot description, xacro)
@@ -1,4 +1,5 @@
 <?xml version="1.0"?>
 <robot name="mascot" xmlns:xacro="http://www.ros.org/wiki/xacro">
+  <static>1</static>
   <xacro:property name="robot_name" value="$(arg robot_name)" />
   <material name="red">
@@ -7,18 +8,18 @@
   <link name="${robot_name}_base_link">
     <inertial>
-      <mass value="1.477" />
-      <origin rpy="1.57 0 0" xyz="0 0 0" />
-      <inertia ixx="0.1152" ixy="0" ixz="0" iyy="0.1152" iyz="0" izz="0.218" />
+      <mass value="0.087" />
+      <origin rpy="0 0 0" xyz="0 0 0" />
+      <inertia ixx="0.1" ixy="0" ixz="0" iyy="0.1" iyz="0" izz="0.1" />
     </inertial>
     <collision name="mascot__collision">
-      <origin rpy="1.57 0 0" xyz="0   0   0.02" />
+      <origin rpy="0 0 0" xyz="0   0   0" />
       <geometry>
-        <mesh scale="0.0005 0.0005 0.0005" filename="package://mascot/meshes/Dji_Tello.stl" />
+        <mesh scale="0.01 0.01 0.01" filename="package://mascot/meshes/DjiTello.dae" />
       </geometry>
     </collision>
     <visual name="mascot__visual">
-      <origin rpy="1.57 0 0" xyz="0   0   0.02" />
+      <origin rpy="0 0 0" xyz="0   0   0" />
       <geometry>
-        <mesh scale="0.0005 0.0005 0.0005" filename="package://mascot/meshes/Dji_Tello.dae" />
+        <mesh scale="0.01 0.01 0.01" filename="package://mascot/meshes/DjiTello.dae" />
       </geometry>
     </visual>
@@ -27,5 +28,5 @@
     <visual>
         <geometry>
-            <sphere radius="0.015"/>
+            <sphere radius="0.0015"/>
         </geometry>
         <material name="red"/>
@@ -35,10 +36,10 @@
     <parent link="${robot_name}_base_link"/>
     <child link="${robot_name}_down_camera_link"/>
-    <origin xyz="-0.06 0 -0.015" rpy="0 1.570796326794897 0"/>
+    <origin xyz="-0.006 0 -0.0015" rpy="0 1.570796326794897 0"/>
   </joint>
   <link name="${robot_name}_front_camera_link">
     <visual>
         <geometry>
-            <sphere radius="0.015"/>
+            <sphere radius="0.0015"/>
         </geometry>
         <material name="red"/>
@@ -48,5 +49,5 @@
     <parent link="${robot_name}_base_link"/>
     <child link="${robot_name}_front_camera_link"/>
-    <origin xyz="0.125 0 0.02" rpy="0 0 0"/>
+    <origin xyz="0.0125 0 0.002" rpy="0 0 0"/>
   </joint>
   <gazebo>
@@ -91,9 +92,9 @@
     </plugin>
   </gazebo>
-  <gazebo reference="${robot_name}_front_camera_link">
+  <!-- <gazebo reference="${robot_name}_front_camera_link">
     <sensor name="${robot_name}_front_camera" type="camera">
       <alwaysOn>true</alwaysOn>
       <visualize>true</visualize>
-      <update_rate>15</update_rate>
+      <update_rate>20</update_rate>
       <camera name="front">
         <horizontal_fov>1.047</horizontal_fov>
@@ -134,5 +135,5 @@
       <alwaysOn>true</alwaysOn>
       <visualize>true</visualize>
-      <update_rate>15</update_rate>
+      <update_rate>20</update_rate>
       <camera name="head">
         <horizontal_fov>1.047</horizontal_fov>
@@ -170,4 +171,8 @@
   </gazebo>
   <gazebo reference="${robot_name}_base_link">
+     <mu1 value="100" />
+      <mu2 value="100" />
+      <kp  value="10000000.0" />
+      <kd  value="1.0" />
      <sensor name='${robot_name}_sensor_sonar' type='sonar'>
       <always_on>1</always_on>
@@ -187,9 +192,14 @@
     </sensor>
   </gazebo>
+  -->
   <gazebo reference="${robot_name}_base_link">
-    <gravity>true</gravity>
+    <!-- <gravity>true</gravity> -->
+    <mu1 value="100" />
+    <mu2 value="100" />
+    <kp  value="10000000.0" />
+    <kd  value="1.0" />
     <sensor name="${robot_name}_imu_sensor" type="imu">
       <always_on>true</always_on>
-      <update_rate>100</update_rate>
+      <update_rate>200</update_rate>
       <visualize>true</visualize>
       <topic>__default_topic__</topic>
@@ -197,5 +207,5 @@
         <topicName>${robot_name}_imu</topicName>
         <bodyName>${robot_name}_base_link</bodyName>
-        <updateRateHZ>10.0</updateRateHZ>
+        <updateRateHZ>200.0</updateRateHZ>
         <gaussianNoise>0.0</gaussianNoise>
         <xyzOffset>0 0 0</xyzOffset>
@@ -207,5 +217,5 @@
     </sensor>
   </gazebo>
-  <gazebo reference="${robot_name}_front_camera_link">
+  <!-- <gazebo reference="${robot_name}_front_camera_link">
     <sensor type="multicamera" name="stereo_camera">
       <update_rate>30.0</update_rate>
@@ -252,5 +262,4 @@
         <cameraInfoTopicName>${robot_name}_camera_info</cameraInfoTopicName>
         <frameName>${robot_name}_front_camera_link</frameName>
-        <!--<rightFrameName>right_camera_optical_frame</rightFrameName>-->
         <hackBaseline>0.07</hackBaseline>
         <distortionK1>0.0</distortionK1>
@@ -261,4 +270,4 @@
       </plugin>
     </sensor>
-  </gazebo>
+  </gazebo> -->
 </robot>

Commit message: add dust

File: urdf/model.xacro (robot description, xacro)
@@ -36,5 +36,5 @@
     <parent link="${robot_name}_base_link"/>
     <child link="${robot_name}_down_camera_link"/>
-    <origin xyz="-0.006 0 -0.0015" rpy="0 1.570796326794897 0"/>
+    <origin xyz="-0.014 0 -0.0065" rpy="0 1.570796326794897 0"/>
   </joint>
   <link name="${robot_name}_front_camera_link">
@@ -49,5 +49,5 @@
     <parent link="${robot_name}_base_link"/>
     <child link="${robot_name}_front_camera_link"/>
-    <origin xyz="0.0125 0 0.002" rpy="0 0 0"/>
+    <origin xyz="0.0285 0 0.0012" rpy="0 0 0"/>
   </joint>
   <gazebo>
@@ -92,5 +92,5 @@
     </plugin>
   </gazebo>
-  <!-- <gazebo reference="${robot_name}_front_camera_link">
+  <gazebo reference="${robot_name}_front_camera_link">
     <sensor name="${robot_name}_front_camera" type="camera">
       <alwaysOn>true</alwaysOn>
@@ -116,5 +116,5 @@
       <plugin name='${robot_name}_front_camera' filename='libgazebo_ros_camera.so'>
         <alwaysOn>true</alwaysOn>
-        <updateRate>0.0</updateRate>
+        <updateRate>20.0</updateRate>
         <cameraName>${robot_name}_front_camera</cameraName>
         <imageTopicName>image_raw</imageTopicName>
@@ -135,5 +135,5 @@
       <alwaysOn>true</alwaysOn>
       <visualize>true</visualize>
-      <update_rate>20</update_rate>
+      <update_rate>30</update_rate>
       <camera name="head">
         <horizontal_fov>1.047</horizontal_fov>
@@ -155,5 +155,5 @@
       <plugin name='${robot_name}_down_camera' filename='libgazebo_ros_camera.so'>
         <alwaysOn>true</alwaysOn>
-        <updateRate>0.0</updateRate>
+        <updateRate>20.0</updateRate>
         <cameraName>${robot_name}_down_camera</cameraName>
         <imageTopicName>image_raw</imageTopicName>
@@ -171,16 +171,12 @@
   </gazebo>
   <gazebo reference="${robot_name}_base_link">
-     <mu1 value="100" />
-      <mu2 value="100" />
-      <kp  value="10000000.0" />
-      <kd  value="1.0" />
      <sensor name='${robot_name}_sensor_sonar' type='sonar'>
       <always_on>1</always_on>
       <visualize>1</visualize>
       <update_rate>100</update_rate>
-      <pose> 0 0 0 0 0 3.141592653 </pose>
+      <pose> 0 0 0 0 0 0 </pose>
       <plugin name='${robot_name}_sonar' filename='libplugin_ros_sonar.so'>
          <topicName>${robot_name}_sonar_sensor</topicName>
-         <frameName>${robot_name}_down_camera_link</frameName>
+         <frameName>${robot_name}_base_link</frameName>
       </plugin>
       <sonar>
@@ -189,10 +185,8 @@
         <radius>0.13974596</radius>
       </sonar>
-      <frame_name>${robot_name}_down_camera_link</frame_name>
-    </sensor>
-  </gazebo>
-  -->
+      <frame_name>${robot_name}_base_link</frame_name>
+    </sensor>
+  </gazebo>
   <gazebo reference="${robot_name}_base_link">
-    <!-- <gravity>true</gravity> -->
     <mu1 value="100" />
     <mu2 value="100" />
@@ -214,5 +208,5 @@
         <initialOrientationAsReference>false</initialOrientationAsReference>
       </plugin>
-      <pose>0 0 0 0 0 0</pose>
+      <pose>-0.014 0 -0.0065 0 0 0</pose>
     </sensor>
   </gazebo>

Commit message: fixed model tello

File: urdf/model.xacro (robot description, xacro)
@@ -15,5 +15,5 @@
       <origin rpy="0 0 0" xyz="0   0   0" />
       <geometry>
-        <mesh scale="0.01 0.01 0.01" filename="package://mascot/meshes/DjiTello.dae" />
+        <mesh scale="1 1 1" filename="package://mascot/meshes/Dji_Tello.stl" />
       </geometry>
     </collision>
@@ -21,5 +21,5 @@
       <origin rpy="0 0 0" xyz="0   0   0" />
       <geometry>
-        <mesh scale="0.01 0.01 0.01" filename="package://mascot/meshes/DjiTello.dae" />
+        <mesh scale="1 1 1" filename="package://mascot/meshes/Dji_Tello.dae" />
       </geometry>
     </visual>
@@ -36,5 +36,5 @@
     <parent link="${robot_name}_base_link"/>
     <child link="${robot_name}_down_camera_link"/>
-    <origin xyz="-0.014 0 -0.0065" rpy="0 1.570796326794897 0"/>
+    <origin xyz="-0.014 0 -0.007" rpy="0 1.570796326794897 0"/>
   </joint>
   <link name="${robot_name}_front_camera_link">
@@ -49,5 +49,5 @@
     <parent link="${robot_name}_base_link"/>
     <child link="${robot_name}_front_camera_link"/>
-    <origin xyz="0.0285 0 0.0012" rpy="0 0 0"/>
+    <origin xyz="0.034 0 0.0012" rpy="0 0 0"/>
   </joint>
   <gazebo>
